Commit message: Changes for new branch

File: body.urdf (robot description, URDF)
Before this commit: robot robot, 2 links, 1 joints
Links:
- added link BackLeg, mass 1; collision box size=0.2 1 0.2; visual box size=0.2 1 0.2
- added link BackLowerLeg, mass 1; collision box size=0.2 0.2 1; visual box size=0.2 0.2 1
- added link FrontLowerLeg, mass 1; collision box size=0.2 0.2 1; visual box size=0.2 0.2 1
- added link LeftLeg, mass 1; collision box size=1 0.2 0.2; visual box size=1 0.2 0.2
- added link LeftLowerLeg, mass 1; collision box size=0.2 0.2 1; visual box size=0.2 0.2 1
- added link RightLeg, mass 1; collision box size=1 0.2 0.2; visual box size=1 0.2 0.2
- added link RightLowerLeg, mass 1; collision box size=0.2 0.2 1; visual box size=0.2 0.2 1
Joints:
- added joint BackLeg_BackLowerLeg: type revolute, parent BackLeg, child BackLowerLeg, origin xyz=0 -1 0 rpy=0 0 0, axis 1 0 0, limit lower=-3.14159 upper=3.14159 effort=0.0 velocity=0.0
- added joint FrontLeg_FrontLowerLeg: type revolute, parent FrontLeg, child FrontLowerLeg, origin xyz=0 1 0 rpy=0 0 0, axis 1 0 0, limit lower=-3.14159 upper=3.14159 effort=0.0 velocity=0.0
- added joint LeftLeg_LeftLowerLeg: type revolute, parent LeftLeg, child LeftLowerLeg, origin xyz=-1 0 0 rpy=0 0 0, axis 0 1 0, limit lower=-3.14159 upper=3.14159 effort=0.0 velocity=0.0
- added joint RightLeg_RightLowerLeg: type revolute, parent RightLeg, child RightLowerLeg, origin xyz=1 0 0 rpy=0 0 0, axis 0 1 0, limit lower=-3.14159 upper=3.14159 effort=0.0 velocity=0.0
- added joint Torso_BackLeg: type revolute, parent Torso, child BackLeg, origin xyz=0 -0.5 1 rpy=0 0 0, axis 1 0 0, limit lower=-3.14159 upper=3.14159 effort=0.0 velocity=0.0
- added joint Torso_LeftLeg: type revolute, parent Torso, child LeftLeg, origin xyz=-0.5 0 1 rpy=0 0 0, axis 0 1 0, limit lower=-3.14159 upper=3.14159 effort=0.0 velocity=0.0
- added joint Torso_RightLeg: type revolute, parent Torso, child RightLeg, origin xyz=0.5 0 1 rpy=0 0 0, axis 0 1 0, limit lower=-3.14159 upper=3.14159 effort=0.0 velocity=0.0

Commit message: First try for rpy rotation

File: body.urdf (robot description, URDF)
Before this commit: robot robot, 2 links, 1 joints
Joints:
- joint s1_s2: origin xyz=0.25 -0.25 0 rpy=0 0 0 -> xyz=0.25 0 0 rpy=0 0 0
